Commit message: feat: migrate to RViz-only simulation, overhaul kinematics, and update documentation

File: src/arm_description/urdf/robot.urdf.xacro (robot description, xacro)
@@ -1,7 +1,42 @@
 <?xml version="1.0"?>
 <robot xmlns:xacro="http://www.ros.org/wiki/xacro" name="decodelabs_arm_workspace">
-  <!-- Include UR5e + Gazebo plugin -->
+  <link name="world"/>
+  <xacro:include filename="$(find arm_description)/urdf/workspace_objects.xacro" />
+  <joint name="world_to_table" type="fixed">
+    <origin xyz="0 0 0" rpy="0 0 0"/>
+    <parent link="world"/>
+    <child link="table_link"/>
+  </joint>
+  <joint name="table_to_l0" type="fixed">
+    <origin xyz="-0.35 0 0.05" rpy="0 0 0"/>
+    <parent link="table_link"/>
+    <child link="l0"/>
+  </joint>
+  <material name="silver">
+    <color rgba="0.9 0.9 0.98 1.0"/>
+  </material>
+  <link name="l0">
+    <inertial>
+      <origin xyz="0.0 0.0 25e-03" rpy="0 0 0"/>
+      <mass value="2e+00"/>
+      <inertia
+        ixx="9.3895308e-03" ixy="0.0" ixz="1.1882474e-03"
+        iyx="0.0" iyy="1.4207390e-02" iyz="9.2874266e-06"
+        izx="1.1882474e-04" izy="9.2874266e-06" izz="1.7661948e-02"/>
+    </inertial>
+    <visual>
+      <geometry>
+        <cylinder radius="0.1" length="0.05"/>
+      </geometry>
+      <origin xyz="0.0 0.0 0.0" rpy="0.0 0.0 0.0"/>
+      <material name="silver"/>
+    </visual>
+  <collision>
+    <geometry>
+      <cylinder radius="0.1" length="0.05"/>
+    </geometry>
+    <origin xyz="0.0 0.0 0.0" rpy="0.0 0.0 0.0"/>
+  </collision>
+ </link>
   <xacro:include filename="$(find arm_description)/urdf/ur5e.urdf.xacro" />
-  <!-- Include Workspace Objects (Table, Cube, Cylinder) -->
-  <xacro:include filename="$(find arm_description)/urdf/workspace_objects.xacro" />
 </robot>

File: src/arm_description/urdf/ur5e.urdf.xacro (robot description, xacro)
@@ -2,9 +2,8 @@
 <robot xmlns:xacro="http://www.ros.org/wiki/xacro" name="decodelabs_ur5e_robot">
   <xacro:include filename="$(find ur_description)/urdf/ur_macro.xacro" />
-  <link name="world"/>
   <xacro:ur_robot
     name="ur5e"
     tf_prefix=""
-    parent="world"
+    parent="l0"
     joint_limits_parameters_file="$(find ur_description)/config/ur5e/joint_limits.yaml"
     kinematics_parameters_file="$(find ur_description)/config/ur5e/default_kinematics.yaml"
@@ -16,14 +15,9 @@
     safety_k_position="20"
     use_fake_hardware="true"
-    fake_sensor_commands="false"
+    fake_sensor_commands="true"
     sim_gazebo="false"
     headless_mode="false"
     >
-    <origin xyz="0 0 0" rpy="0 0 0" />
+    <origin xyz="0 0 0.025" rpy="0 0 0" />
   </xacro:ur_robot>
-  <gazebo>
-    <plugin filename="libgazebo_ros2_control.so" name="gazebo_ros2_control">
-      <parameters>$(find arm_control)/config/controllers.yaml</parameters>
-    </plugin>
-  </gazebo>
 </robot>

File: src/arm_description/urdf/workspace_objects.xacro (robot description, xacro)
@@ -1,9 +1,8 @@
 <?xml version="1.0"?>
 <robot xmlns:xacro="http://www.ros.org/wiki/xacro" name="workspace_objects">
-  <!-- Table: 1.0m x 0.6m x 0.05m, positioned below robot -->
   <link name="table_link">
     <visual>
       <geometry><box size="1.0 0.6 0.05"/></geometry>
-      <origin xyz="0.5 0.0 -0.025" rpy="0 0 0"/>
+      <origin xyz="0 0 0" rpy="0 0 0"/>
       <material name="brown">
         <color rgba="0.6 0.4 0.2 1.0"/>
@@ -12,5 +11,5 @@
     <collision>
       <geometry><box size="1.0 0.6 0.05"/></geometry>
-      <origin xyz="0.5 0.0 -0.025" rpy="0 0 0"/>
+      <origin xyz="0 0 0" rpy="0 0 0"/>
     </collision>
     <inertial>
@@ -19,15 +18,5 @@
     </inertial>
   </link>
-  <joint name="base_link_to_table" type="fixed">
-    <parent link="base_link"/>
-    <child link="table_link"/>
-    <origin xyz="0 0 -0.5" rpy="0 0 0"/>
-  </joint>
-  <!-- Gazebo material for table -->
-  <gazebo reference="table_link">
-    <material>Gazebo/Wood</material>
-    <static>true</static>
-  </gazebo>
-  <!-- Cube 1: 0.05m x 0.05m x 0.05m, at (0.4, 0.2, 0.025) -->
+  <!-- Cube 1: on table at (0.0, 0.15, 0.05) relative to table center -->
   <link name="cube_1_link">
     <visual>
@@ -47,13 +36,10 @@
     </inertial>
   </link>
-  <joint name="base_link_to_cube_1" type="fixed">
-    <parent link="base_link"/>
+  <joint name="table_to_cube_1" type="fixed">
+    <parent link="table_link"/>
     <child link="cube_1_link"/>
-    <origin xyz="0.4 0.2 -0.475" rpy="0 0 0"/>
+    <origin xyz="0.0 0.15 0.05" rpy="0 0 0"/>
   </joint>
-  <gazebo reference="cube_1_link">
-    <material>Gazebo/Red</material>
-  </gazebo>
-  <!-- Cylinder 1: radius 0.025m, height 0.1m, at (0.4, -0.2, 0.05) -->
+  <!-- Cylinder 1: on table at (0.0, -0.15, 0.075) relative to table center -->
   <link name="cylinder_1_link">
     <visual>
@@ -73,11 +59,8 @@
     </inertial>
   </link>
-  <joint name="base_link_to_cylinder_1" type="fixed">
-    <parent link="base_link"/>
+  <joint name="table_to_cylinder_1" type="fixed">
+    <parent link="table_link"/>
     <child link="cylinder_1_link"/>
-    <origin xyz="0.4 -0.2 -0.45" rpy="0 0 0"/>
+    <origin xyz="0.0 -0.15 0.075" rpy="0 0 0"/>
   </joint>
-  <gazebo reference="cylinder_1_link">
-    <material>Gazebo/Blue</material>
-  </gazebo>
 </robot>
